Commit message: Hardware Interface

File: src/myroboticarm_description_cpp/urdf/myroboticarm.urdf.xacro (robot description, xacro)
@@ -1,4 +1,5 @@
 <?xml version="1.0"?>
 <robot  xmlns:xacro="http://www.ros.org/wiki/xacro" name="my_robotic_arm">
+    <xacro:arg name="is_sim" default="true"/>
     <xacro:arg name="is_ignition" default="true"/>
     <xacro:include filename="$(find myroboticarm_description_cpp)/urdf/myroboticarm_gazebo.xacro"/>
@@ -175,7 +176,4 @@
                 <mesh filename="package://myroboticarm_description_cpp/meshes/pi_camera.STL" scale="0.01 0.01 0.01"/>
             </geometry>
-<!--            <material name="CameraBlue">
-                <color rgba="0 0 1 1"/>
-            </material>-->
         </visual>
         <collision>
@@ -191,57 +189,3 @@
         <origin xyz="0.0 0.1 0.1" rpy="0 0 0"/>
     </joint>
-<!--   <gazebo reference="rgb_camera">
-        <sensor type="camera" name="rgb_camera">
-            <update_rate>30.0</update_rate>
-            <camera>
-                <horizontal_fov>1.15</horizontal_fov>
-                <vertical_fov>0.71</vertical_fov>
-                <image>
-                    <width>2304</width>
-                    <height>1296</height>
-                    <format>R8G8B8</format>
-                </image>
-            </camera>
-            <plugin name="gazebo_camera_controller" filename="libgazebo_ros_camera.so">
-                <camera_name>rgb_camera</camera_name>
-                <image_topic_name>image_raw</image_topic_name>
-                <camera_info_topic_name>camera_info</camera_info_topic_name>
-                <frame_name>rgb_camera</frame_name>
-            </plugin>
-        </sensor>
-    </gazebo> -->
-<!--    <gazebo>
-        <plugin name="camera_controller" filename="libgazebo_ros_camera.so">
-            <camera_name>camera</camera_name>
-            <image_topic_name>image_raw</image_topic_name>
-            <camera_info_topic_name>camera_info</camera_info_topic_name>
-            <frame_name>rgb_camera</frame_name>
-            <gz_frame_id>rgb_camera</gz_frame_id>
-        </plugin>
-    </gazebo>
-    <gazebo reference="rgb_camera">
-        <sensor name="camera" type="camera">
-            <always_on>true</always_on>
-            <update_rate>30.0</update_rate>
-            <visualize>true</visualize>
-            <topic>image_raw</topic>
-            <gz_frame_id>rgb_camera</gz_frame_id>
-            <camera name="camera">
-                <horizontal_fov>1.21126</horizontal_fov>
-                <image>
-                    <width>2304</width>
-                    <height>1296</height>
-                    <format>R8G8B8</format>
-                </image>
-                <distortion>
-                    <k1>0.0</k1>
-                    <k2>0.0</k2>
-                    <k3>0.0</k3>
-                    <p1>0.0</p1>
-                    <p2>0.0</p2>
-                    <center>0.5 0.5</center>
-                </distortion>
-            </camera>
-        </sensor>
-    </gazebo>       -->
 </robot>

File: src/myroboticarm_description_cpp/urdf/myroboticarm_ros2_control.xacro (robot description, xacro)
@@ -3,8 +3,24 @@
     <ros2_control name="RobotSystem"  type="system">
         <xacro:property name="PI" value="3.14159265359" />
-        <xacro:if value="$(arg is_ignition)">
+        <xacro:if value= "$(arg is_sim)">
             <hardware>
-                <plugin>
-                    ign_ros2_control/IgnitionSystem</plugin>
+                <plugin>gazebo_ros2_control/GazeboSystem</plugin>
+            </hardware>
+          <joint name="joint_5">
+            <param name="mimic">joint_4</param>
+            <param name="multiplier">-1</param>
+            <state_interface name="position"/>
+            <state_interface name="velocity"/>
+          </joint>
+        </xacro:if>
+        <xacro:unless value= "$(arg is_sim)">
+            <hardware>
+                <plugin>myroboticarm_controller/MyroboticarmInterface</plugin>
+                <param name="port">/dev/ttyUSB0</param>
+            </hardware>
+        </xacro:unless>
+        <!-- <xacro:if value="$(arg is_ignition)">
+            <hardware>
+                <plugin>ign_ros2_control/IgnitionSystem</plugin>
                 <plugin>mock_components/GenericSystem</plugin>
             </hardware>
@@ -16,5 +32,5 @@
                 <plugin>gazebo_ros2_control/GazeboSystem</plugin>
             </hardware>
-        </xacro:unless>
+        </xacro:unless>  -->
         <joint name="joint_1">
             <command_interface name="position">
@@ -49,8 +65,4 @@
             <state_interface name="velocity"/>
         </joint>
-        <joint name="joint_5">
-            <param name="mimic">joint_4</param>
-            <param name="multiplier">-1</param>
-        </joint>
     </ros2_control>
 </robot>
